File: hardware/v1/schematics/sensof_ht.sch (KiCad schematic (older format))
At the start: 23 parts, among them J1 Conn_01x06, J2 Conn_01x04, U1 Si4010-GT, U2 HTU21D/Si7020

Commit message: HW: Updated V1 schematic to KiCad 5.0
Parts:
- AE1: symbol Antenna -> Device:Antenna
- BT1: value Battery_Cell -> CR2032; symbol Battery_Cell -> Device:Battery_Cell
- C1, C10, C2, C3, C4, C5, C6, C7, C8, C9: symbol C -> Device:C
- J1: symbol Conn_01x06 -> Connector_Generic:Conn_01x06
- J2: symbol Conn_01x04 -> Connector_Generic:Conn_01x04
- L1, L2, L3, L4, L5: symbol L -> Device:L
- R1, R2: symbol R -> Device:R
- U1: symbol Si4010-GT -> si4010:Si4010-GT
- U2: symbol HTU21D -> htu21d:HTU21D
