File: hardware/v1/schematics/sensof_ht.sch (KiCad schematic (older format))
At the start: 23 parts, among them J1 Conn_01x06, J2 Conn_01x04, U1 Si4010-GT, U2 HTU21D/Si7020

Commit message: HW: Change part suggestions to the once I actually used in the prototype
Parts:
- C2, C4: Mfr. No GRM1555C1E6R8BA01D -> GJM1555C1H6R8CB01D; Mouser No 81-GRM1555C1E6R8BA1D -> 81-GJM1555C1H6R8CB01
- C3: Mfr. No GRM1555C1E4R3BA01D -> GJM1555C1H4R3BB01D; Mouser No 81-GRM1555C1E4R3BA1D -> 81-GJM1555C1H4R3BB01
- C5: Mfr. No GRM1555C1H2R7BA01D -> GJM1555C1H2R7BB01D; Mouser No 81-GRM1555C1H2R7BA1D -> 81-GJM1555C1H2R7BB01
- C6: Mfr. No GRM1555C1H1R8WA01D -> GJM1555C1H1R8WB01D; Mouser No 81-GRM1555C1H1R8WA1D -> 81-GJM1555C1H1R8WB1D
- C8: Mfr. No GRM1555C1H102JA01D -> GCM155L81H102KA37D; Mouser No 81-GRM1555C1H102JA1D -> 81-GCM155L81H102KA7D
- L3, L4: Mfr. No LQW15AN16NJ80D -> LQW15AN16NJ00D; Mouser No 81-LQW15AN16NJ80D -> 81-LQW15AN16NJ00D
Changed lines of the file:
@@
 F 3 "" H 3350 3700 50  0001 C CNN
 F 4 "Murata" H 0   0   50  0001 C CNN "Manufacturer"
-F 5 "GRM1555C1H2R7BA01D" H 0   0   50  0001 C CNN "Mfr. No"
-F 6 "81-GRM1555C1H2R7BA1D" H 0   0   50  0001 C CNN "Mouser No"
+F 5 "GJM1555C1H2R7BB01D" H 0   0   50  0001 C CNN "Mfr. No"
+F 6 "81-GJM1555C1H2R7BB01" H 0   0   50  0001 C CNN "Mouser No"
 F 7 "±5%; C0G (based on 4010-DKPB434-BM_BOM.xls)" H 0   0   50  0001 C CNN "Note"
 	1    3350 3700
@@
 F 3 "" H 2500 2950 50  0001 C CNN
 F 4 "Murata" H 0   0   50  0001 C CNN "Manufacturer"
-F 5 "GRM1555C1E4R3BA01D" H 0   0   50  0001 C CNN "Mfr. No"
-F 6 "81-GRM1555C1E4R3BA1D" H 0   0   50  0001 C CNN "Mouser No"
+F 5 "GJM1555C1H4R3BB01D" H 0   0   50  0001 C CNN "Mfr. No"
+F 6 "81-GJM1555C1H4R3BB01" H 0   0   50  0001 C CNN "Mouser No"
 F 7 "±5%; C0G (based on 4010-DKPB434-BM_BOM.xls)" H 0   0   50  0001 C CNN "Note"
 	1    2500 2950
@@
 F 3 "" H 2150 4500 50  0001 C CNN
 F 4 "Murata" H 0   0   50  0001 C CNN "Manufacturer"
-F 5 "GRM1555C1E6R8BA01D" H 0   0   50  0001 C CNN "Mfr. No"
-F 6 "81-GRM1555C1E6R8BA1D" H 0   0   50  0001 C CNN "Mouser No"
+F 5 "GJM1555C1H6R8CB01D" H 0   0   50  0001 C CNN "Mfr. No"
+F 6 "81-GJM1555C1H6R8CB01" H 0   0   50  0001 C CNN "Mouser No"
 F 7 "±5%; C0G (based on 4010-DKPB434-BM_BOM.xls)" H 0   0   50  0001 C CNN "Note"
 	1    2150 4500
@@
 F 3 "" H 2750 4500 50  0001 C CNN
 F 4 "Murata" H 0   0   50  0001 C CNN "Manufacturer"
-F 5 "GRM1555C1E6R8BA01D" H 0   0   50  0001 C CNN "Mfr. No"
-F 6 "81-GRM1555C1E6R8BA1D" H 0   0   50  0001 C CNN "Mouser No"
+F 5 "GJM1555C1H6R8CB01D" H 0   0   50  0001 C CNN "Mfr. No"
+F 6 "81-GJM1555C1H6R8CB01" H 0   0   50  0001 C CNN "Mouser No"
 F 7 "±5%; C0G (based on 4010-DKPB434-BM_BOM.xls)" H 0   0   50  0001 C CNN "Note"
 	1    2750 4500
@@
 F 3 "" H 3400 4250 50  0001 C CNN
 F 4 "Murata" H 0   0   50  0001 C CNN "Manufacturer"
-F 5 "GRM1555C1H1R8WA01D" H 0   0   50  0001 C CNN "Mfr. No"
-F 6 "81-GRM1555C1H1R8WA1D" H 0   0   50  0001 C CNN "Mouser No"
+F 5 "GJM1555C1H1R8WB01D" H 0   0   50  0001 C CNN "Mfr. No"
+F 6 "81-GJM1555C1H1R8WB1D" H 0   0   50  0001 C CNN "Mouser No"
 F 7 "±5%; C0G (based on 4010-DKPB434-BM_BOM.xls)" H 0   0   50  0001 C CNN "Note"
 	1    3400 4250
@@
 F 3 "" H 3700 3750 50  0001 C CNN
 F 4 "Murata" H 0   0   50  0001 C CNN "Manufacturer"
-F 5 "LQW15AN16NJ80D" H 0   0   50  0001 C CNN "Mfr. No"
-F 6 "81-LQW15AN16NJ80D" H 0   0   50  0001 C CNN "Mouser No"
+F 5 "LQW15AN16NJ00D" H 0   0   50  0001 C CNN "Mfr. No"
+F 6 "81-LQW15AN16NJ00D" H 0   0   50  0001 C CNN "Mouser No"
 F 7 "See sensof_ht-BOM.ods:‘Inductor Selection’ tab" H 0   0   50  0001 C CNN "Note"
 	1    3700 3750
@@
 F 3 "" H 3700 3350 50  0001 C CNN
 F 4 "Murata" H 0   0   50  0001 C CNN "Manufacturer"
-F 5 "LQW15AN16NJ80D" H 0   0   50  0001 C CNN "Mfr. No"
-F 6 "81-LQW15AN16NJ80D" H 0   0   50  0001 C CNN "Mouser No"
+F 5 "LQW15AN16NJ00D" H 0   0   50  0001 C CNN "Mfr. No"
+F 6 "81-LQW15AN16NJ00D" H 0   0   50  0001 C CNN "Mouser No"
 F 7 "See sensof_ht-BOM.ods:‘Inductor Selection’ tab" H 0   0   50  0001 C CNN "Note"
 	1    3700 3350
@@
 F 5 "885012106018" H 0   0   50  0001 C CNN "Mfr. No"
 F 6 "710-885012106018" H 0   0   50  0001 C CNN "Mouser No"
+F 7 "" H 0   0   50  0001 C CNN "Note"
 	1    5600 2250
 	1    0    0    -1
@@
 F 3 "" H 5850 2250 50  0001 C CNN
 F 4 "Murata" H 0   0   50  0001 C CNN "Manufacturer"
-F 5 "GRM1555C1H102JA01D" H 0   0   50  0001 C CNN "Mfr. No"
-F 6 "81-GRM1555C1H102JA1D" H 0   0   50  0001 C CNN "Mouser No"
+F 5 "GCM155L81H102KA37D" H 0   0   50  0001 C CNN "Mfr. No"
+F 6 "81-GCM155L81H102KA7D" H 0   0   50  0001 C CNN "Mouser No"
+F 7 "" H 0   0   50  0001 C CNN "Note"
 	1    5850 2250
 	1    0    0    -1
@@
 F 5 "GRM1555C1H271JA01J" H 0   0   50  0001 C CNN "Mfr. No"
 F 6 "81-GRM1555C1H271JA1J" H 0   0   50  0001 C CNN "Mouser No"
+F 7 "" H 0   0   50  0001 C CNN "Note"
 	1    6100 2250
 	1    0    0    -1
@@
 F 5 "SI7020-A20-GM1" H 0   0   50  0001 C CNN "Mfr. No"
 F 6 "634-SI7020-A20-GM1" H 0   0   50  0001 C CNN "Mouser No"
+F 7 "" H 0   0   50  0001 C CNN "Note"
 	1    8700 3400
 	1    0    0    -1
@@
 F 5 "CRCW040210K0FKEDC" H 0   0   50  0001 C CNN "Mfr. No"
 F 6 "71-CRCW040210K0FKEDC" H 0   0   50  0001 C CNN "Mouser No"
+F 7 "" H 0   0   50  0001 C CNN "Note"
 	1    7650 3050
 	1    0    0    -1
@@
 F 5 "CRCW040210K0FKEDC" H 0   0   50  0001 C CNN "Mfr. No"
 F 6 "71-CRCW040210K0FKEDC" H 0   0   50  0001 C CNN "Mouser No"
+F 7 "" H 0   0   50  0001 C CNN "Note"
 	1    7350 3050
 	1    0    0    -1
@@
 F 5 "PRT-10210" H 0   0   50  0001 C CNN "Mfr. No"
 F 6 "474-PRT-10210" H 0   0   50  0001 C CNN "Mouser No"
+F 7 "" H 0   0   50  0001 C CNN "Note"
 	1    6400 4550
 	0    -1   1    0
@@
 F 2 "Abracon_ACAG1204-433-T:ACAG1204-433-T" H 1500 3900 50  0001 C CNN
 F 3 "" H 1500 3900 50  0001 C CNN
+F 4 "" H 0   0   50  0001 C CNN "Note"
 	1    1500 3900
 	1    0    0    -1
@@
 F 2 "Linx_BAT-HLD-001:Linx_BAT-HLD-001" V 9650 4810 50  0001 C CNN
 F 3 "" V 9650 4810 50  0001 C CNN
+F 4 "" H 0   0   50  0001 C CNN "Note"
 	1    9650 4750
 	1    0    0    -1
@@
 F 5 "885012105016" H 0   0   50  0001 C CNN "Mfr. No"
 F 6 "710-885012105016" H 0   0   50  0001 C CNN "Mouser No"
+F 7 "" H 0   0   50  0001 C CNN "Note"
 	1    8900 2700
 	1    0    0    -1
@@
 F 2 "Connectors_JST:JST_SH_SM04B-SRSS-TB_04x1.00mm_Angled" H 8000 4850 50  0001 C CNN
 F 3 "" H 8000 4850 50  0001 C CNN
+F 4 "" H 0   0   50  0001 C CNN "Note"
 	1    8000 4850
 	0    -1   1    0
@@
 F 5 "SI4010-C2-GT" H 0   0   50  0001 C CNN "Mfr. No"
 F 6 "634-SI4010-C2-GT" H 0   0   50  0001 C CNN "Mouser No"
+F 7 "" H 0   0   50  0001 C CNN "Note"
 	1    5400 3550
 	1    0    0    -1
