File: hardware/v2/schematics/sensof_ht.sch (KiCad schematic (older format))
At the start: 20 parts, among them U1 Si4010-GS, U2 HTU21D/Si7020

Commit message: HW: PCBv2 Upgraded to KiCad 5.0 and switch to shared component library
Parts:
- BT1: symbol Battery_Cell -> Device:Battery_Cell
- C1, C2, C3, C4, C5, C6: symbol C -> Device:C
- L1: symbol L -> Device:L
- R1, R2: symbol R -> Device:R
- TP1, TP2, TP3, TP4, TP5, TP6, TP7, TP8: symbol TEST_1P -> Connector:TestPoint
- U1: symbol Si4010-GS -> si4010:Si4010-GS
- U2: symbol HTU21D -> Sensor_Humidity:Si7020-A20
Connections:
- wire segments 71 -> 83
- no-connect marks 4 -> 5
Other:
- moved on the sheet: C3, C4, C5, C6, R1, R2, U1

Commit message: PCBv2: Add part numbers to schematic
Added part numbers from BOM to schematic.
Parts:
- BT1: Manufacturer (none) -> Linx Technologies; Mfr. No (none) -> BAT-HLD-001; Mouser No (none) -> 712-BAT-HLD-001
- C1: Manufacturer (none) -> Murata; Mfr. No (none) -> GJM1555C1H2R7BB01D; Mouser No (none) -> 81-GJM1555C1H2R7BB01
- C2, TP1, TP2, TP3, TP4, TP5, TP6, TP7, TP8: Manufacturer (none) -> -; Mfr. No (none) -> -; Mouser No (none) -> -
- C3: Manufacturer (none) -> Taiyo Yuden; Mfr. No (none) -> LMK107BJ225KAHT; Mouser No (none) -> 963-LMK107BJ225KAHT
- C4: Manufacturer (none) -> KEMET; Mfr. No (none) -> C0603C102J5RACTU; Mouser No (none) -> 80-C0603C102J5R
- C5: Manufacturer (none) -> Yageo; Mfr. No (none) -> CC0603JRX7R9BB271; Mouser No (none) -> 603-CC603JRX7R9BB271
- C6: Manufacturer (none) -> Yageo; Mfr. No (none) -> CC0603KRX7R6BB104; Mouser No (none) -> 603-CC603KRX7R6BB104
- L1: Manufacturer (none) -> Murata; Mfr. No (none) -> LQW15CNR22J10D; Mouser No (none) -> 81-LQW15CNR22J10D
- R1, R2: Manufacturer (none) -> Yageo; Mfr. No (none) -> RE0603FRE0710KL; Mouser No (none) -> 603-RE0603FRE0710KL
- U1: Manufacturer (none) -> Silicon Labs; Mfr. No (none) -> SI4010-C2-GS; Mouser No (none) -> 634-SI4010-C2-GS
- U2: Manufacturer (none) -> TE Connectivity; Mfr. No (none) -> HTU21DF; Mouser No (none) -> 824-HPP845E131R5
Changed lines of the file:
@@
 Sheet 1 1
 Title "Sensof HT v2"
-Date "2018-09-13"
+Date "2018-09-16"
 Rev "01"
 Comp "Copyright (c) 2018, David Imhoff <dimhoff.devel@gmail.com>"
@@
 F 2 "silabs_0402:C_0402" H 3338 3550 50  0001 C CNN
 F 3 "" H 3300 3700 50  0001 C CNN
+F 4 "Murata" H 0   0   50  0001 C CNN "Manufacturer"
+F 5 "GJM1555C1H2R7BB01D" H 0   0   50  0001 C CNN "Mfr. No"
+F 6 "81-GJM1555C1H2R7BB01" H 0   0   50  0001 C CNN "Mouser No"
 	1    3300 3700
 	-1   0    0    1
@@
 F 2 "silabs_0402:C_0402" H 3300 3300 50  0001 C CNN
 F 3 "" H 3300 3300 50  0001 C CNN
+F 4 "Murata" H 0   0   50  0001 C CNN "Manufacturer"
+F 5 "LQW15CNR22J10D" H 0   0   50  0001 C CNN "Mfr. No"
+F 6 "81-LQW15CNR22J10D" H 0   0   50  0001 C CNN "Mouser No"
 	1    3300 3300
 	1    0    0    -1
@@
 F 2 "Capacitors_SMD:C_0603" H 5538 2200 50  0001 C CNN
 F 3 "" H 5500 2350 50  0001 C CNN
+F 4 "Taiyo Yuden" H 0   0   50  0001 C CNN "Manufacturer"
+F 5 "LMK107BJ225KAHT" H 0   0   50  0001 C CNN "Mfr. No"
+F 6 "963-LMK107BJ225KAHT" H 0   0   50  0001 C CNN "Mouser No"
 	1    5500 2350
 	1    0    0    -1
@@
 F 2 "Capacitors_SMD:C_0603" H 5788 2200 50  0001 C CNN
 F 3 "" H 5750 2350 50  0001 C CNN
+F 4 "KEMET" H 0   0   50  0001 C CNN "Manufacturer"
+F 5 "C0603C102J5RACTU" H 0   0   50  0001 C CNN "Mfr. No"
+F 6 "80-C0603C102J5R" H 0   0   50  0001 C CNN "Mouser No"
 	1    5750 2350
 	1    0    0    -1
@@
 F 2 "Capacitors_SMD:C_0603" H 6038 2200 50  0001 C CNN
 F 3 "" H 6000 2350 50  0001 C CNN
+F 4 "Yageo" H 0   0   50  0001 C CNN "Manufacturer"
+F 5 "CC0603JRX7R9BB271" H 0   0   50  0001 C CNN "Mfr. No"
+F 6 "603-CC603JRX7R9BB271" H 0   0   50  0001 C CNN "Mouser No"
 	1    6000 2350
 	1    0    0    -1
@@
 F 2 "Housings_DFN_QFN:DFN-6-1EP_3x3mm_Pitch0.95mm" H 8050 3400 60  0001 C CNN
 F 3 "" H 8050 3400 60  0001 C CNN
+F 4 "TE Connectivity" H 0   0   50  0001 C CNN "Manufacturer"
+F 5 "HTU21DF" H 0   0   50  0001 C CNN "Mfr. No"
+F 6 "824-HPP845E131R5" H 0   0   50  0001 C CNN "Mouser No"
 	1    8050 3400
 	1    0    0    -1
@@
 F 2 "Resistors_SMD:R_0603" V 6930 3050 50  0001 C CNN
 F 3 "" H 7000 3050 50  0001 C CNN
+F 4 "Yageo" H 0   0   50  0001 C CNN "Manufacturer"
+F 5 "RE0603FRE0710KL" H 0   0   50  0001 C CNN "Mfr. No"
+F 6 "603-RE0603FRE0710KL" H 0   0   50  0001 C CNN "Mouser No"
 	1    7000 3050
 	1    0    0    -1
@@
 F 2 "Resistors_SMD:R_0603" V 6630 3050 50  0001 C CNN
 F 3 "" H 6700 3050 50  0001 C CNN
+F 4 "Yageo" H 0   0   50  0001 C CNN "Manufacturer"
+F 5 "RE0603FRE0710KL" H 0   0   50  0001 C CNN "Mfr. No"
+F 6 "603-RE0603FRE0710KL" H 0   0   50  0001 C CNN "Mouser No"
 	1    6700 3050
 	1    0    0    -1
@@
 F 2 "silabs_cr2032:silabs_cr2032" V 3750 4960 50  0001 C CNN
 F 3 "" V 3750 4960 50  0001 C CNN
+F 4 "Linx Technologies" H 0   0   50  0001 C CNN "Manufacturer"
+F 5 "BAT-HLD-001" H 0   0   50  0001 C CNN "Mfr. No"
+F 6 "712-BAT-HLD-001" H 0   0   50  0001 C CNN "Mouser No"
 	1    3750 4900
 	1    0    0    -1
@@
 F 2 "Capacitors_SMD:C_0603" H 8388 2600 50  0001 C CNN
 F 3 "" H 8350 2750 50  0001 C CNN
+F 4 "Yageo" H 0   0   50  0001 C CNN "Manufacturer"
+F 5 "CC0603KRX7R6BB104" H 0   0   50  0001 C CNN "Mfr. No"
+F 6 "603-CC603KRX7R6BB104" H 0   0   50  0001 C CNN "Mouser No"
 	1    8350 2750
 	1    0    0    -1
@@
 F 2 "Capacitors_SMD:C_0603" H 4038 3350 50  0001 C CNN
 F 3 "" H 4000 3500 50  0001 C CNN
+F 4 "-" H 0   0   50  0001 C CNN "Manufacturer"
+F 5 "-" H 0   0   50  0001 C CNN "Mfr. No"
+F 6 "-" H 0   0   50  0001 C CNN "Mouser No"
 	1    4000 3500
 	-1   0    0    1
@@
 F 2 "Measurement_Point_Round-SMD-Pad_Small-Labeled:Measurement_Point_Round-SMD-Pad_Small-Labeled" H 7800 4150 50  0001 C CNN
 F 3 "" H 7800 4150 50  0001 C CNN
+F 4 "-" H 0   0   50  0001 C CNN "Manufacturer"
+F 5 "-" H 0   0   50  0001 C CNN "Mfr. No"
+F 6 "-" H 0   0   50  0001 C CNN "Mouser No"
 	1    7600 4150
 	0    1    1    0
@@
 F 2 "Measurement_Point_Round-SMD-Pad_Small-Labeled:Measurement_Point_Round-SMD-Pad_Small-Labeled" H 7800 4300 50  0001 C CNN
 F 3 "" H 7800 4300 50  0001 C CNN
+F 4 "-" H 0   0   50  0001 C CNN "Manufacturer"
+F 5 "-" H 0   0   50  0001 C CNN "Mfr. No"
+F 6 "-" H 0   0   50  0001 C CNN "Mouser No"
 	1    7600 4300
 	0    1    1    0
@@
 F 2 "Measurement_Point_Round-SMD-Pad_Small-Labeled:Measurement_Point_Round-SMD-Pad_Small-Labeled" H 7800 4450 50  0001 C CNN
 F 3 "" H 7800 4450 50  0001 C CNN
+F 4 "-" H 0   0   50  0001 C CNN "Manufacturer"
+F 5 "-" H 0   0   50  0001 C CNN "Mfr. No"
+F 6 "-" H 0   0   50  0001 C CNN "Mouser No"
 	1    7600 4450
 	0    1    1    0
@@
 F 2 "Measurement_Point_Round-SMD-Pad_Small-Labeled:Measurement_Point_Round-SMD-Pad_Small-Labeled" H 7800 4600 50  0001 C CNN
 F 3 "" H 7800 4600 50  0001 C CNN
+F 4 "-" H 0   0   50  0001 C CNN "Manufacturer"
+F 5 "-" H 0   0   50  0001 C CNN "Mfr. No"
+F 6 "-" H 0   0   50  0001 C CNN "Mouser No"
 	1    7600 4600
 	0    1    1    0
@@
 F 2 "Measurement_Point_Round-SMD-Pad_Small-Labeled:Measurement_Point_Round-SMD-Pad_Small-Labeled" H 7800 4750 50  0001 C CNN
 F 3 "" H 7800 4750 50  0001 C CNN
+F 4 "-" H 0   0   50  0001 C CNN "Manufacturer"
+F 5 "-" H 0   0   50  0001 C CNN "Mfr. No"
+F 6 "-" H 0   0   50  0001 C CNN "Mouser No"
 	1    7600 4750
 	0    1    1    0
@@
 F 2 "Measurement_Point_Round-SMD-Pad_Small-Labeled:Measurement_Point_Round-SMD-Pad_Small-Labeled" H 7800 4900 50  0001 C CNN
 F 3 "" H 7800 4900 50  0001 C CNN
+F 4 "-" H 0   0   50  0001 C CNN "Manufacturer"
+F 5 "-" H 0   0   50  0001 C CNN "Mfr. No"
+F 6 "-" H 0   0   50  0001 C CNN "Mouser No"
 	1    7600 4900
 	0    1    1    0
@@
 F 2 "Measurement_Point_Round-SMD-Pad_Small-Labeled:Measurement_Point_Round-SMD-Pad_Small-Labeled" H 7800 5050 50  0001 C CNN
 F 3 "" H 7800 5050 50  0001 C CNN
+F 4 "-" H 0   0   50  0001 C CNN "Manufacturer"
+F 5 "-" H 0   0   50  0001 C CNN "Mfr. No"
+F 6 "-" H 0   0   50  0001 C CNN "Mouser No"
 	1    7600 5050
 	0    1    1    0
@@
 F 2 "Measurement_Point_Round-SMD-Pad_Small-Labeled:Measurement_Point_Round-SMD-Pad_Small-Labeled" H 7800 5200 50  0001 C CNN
 F 3 "" H 7800 5200 50  0001 C CNN
+F 4 "-" H 0   0   50  0001 C CNN "Manufacturer"
+F 5 "-" H 0   0   50  0001 C CNN "Mfr. No"
+F 6 "-" H 0   0   50  0001 C CNN "Mouser No"
 	1    7600 5200
 	0    1    1    0
@@
 F 2 "Housings_SOIC:SOIC-14_3.9x8.7mm_Pitch1.27mm" H 5400 3000 60  0001 C CNN
 F 3 "" H 5400 3000 60  0001 C CNN
+F 4 "Silicon Labs" H 5350 3550 50  0001 C CNN "Manufacturer"
+F 5 "SI4010-C2-GS" H 5350 3550 50  0001 C CNN "Mfr. No"
+F 6 "634-SI4010-C2-GS" H 5350 3550 50  0001 C CNN "Mouser No"
 	1    5350 3550
 	1    0    0    -1

Commit message: PCBv2: Add part requirements to schematic
Parts:
- C1: Requirements (none) -> ±5%; C0G (based on 4010-DKMX-434_BOM.xls)
- L1: Requirements (none) -> Coilcraft 0402HP-220NX_LU
Changed lines of the file:
@@
 F 5 "GJM1555C1H2R7BB01D" H 0   0   50  0001 C CNN "Mfr. No"
 F 6 "81-GJM1555C1H2R7BB01" H 0   0   50  0001 C CNN "Mouser No"
+F 7 "±5%; C0G (based on 4010-DKMX-434_BOM.xls)" H 3300 3700 50  0001 C CNN "Requirements"
 	1    3300 3700
 	-1   0    0    1
@@
 F 5 "LQW15CNR22J10D" H 0   0   50  0001 C CNN "Mfr. No"
 F 6 "81-LQW15CNR22J10D" H 0   0   50  0001 C CNN "Mouser No"
+F 7 "Coilcraft 0402HP-220NX_LU" H 3300 3300 50  0001 C CNN "Requirements"
 	1    3300 3300
 	1    0    0    -1
